Commit message: practice

File: src/ur5_robot_moveit_config/config/ur5_robot.ros2_control.xacro (robot description, xacro)
@@ -2,5 +2,5 @@
 <robot xmlns:xacro="http://www.ros.org/wiki/xacro">
     <xacro:macro name="ur5_robot_ros2_control" params="name initial_positions_file">
-        <xacro:property name="initial_positions" value="${load_yaml(initial_positions_file)['initial_positions']}"/>
+        <xacro:property name="initial_positions" value="${xacro.load_yaml(initial_positions_file)['initial_positions']}"/>
         <ros2_control name="${name}" type="system">
             <hardware>

File: src/ur5_robot_moveit_config/config/ur5_robot.urdf.xacro (robot description, xacro)
@@ -5,5 +5,10 @@
     <xacro:include filename="$(find ur_description)/urdf/ur5.xacro" />
     <!-- Import control_xacro -->
-    <xacro:include filename="ur5_robot.ros2_control.xacro" />
+    <xacro:include filename="$(find ur5_robot_moveit_config)/config/ur5_robot.ros2_control.xacro" />
     <xacro:ur5_robot_ros2_control name="FakeSystem" initial_positions_file="$(arg initial_positions_file)"/>
+    <gazebo>
+      <plugin filename="libgazebo_ros2_control.so" name="gazebo_ros2_control">
+        <parameters>$(find ur5_robot_moveit_config)/config/ros2_controllers.yaml</parameters>
+      </plugin>
+    </gazebo>
 </robot>
